Commit message: Finished simulation and PID controllers settings.

File: Simulation/src/manipulator/urdf/manipulator.urdf (robot description, URDF)
Before this commit: robot manipulator, 8 links, 7 joints
Joints:
- joint arm_rotation: limit lower=-2.5 upper=0 effort=50 velocity=0.25 -> lower=-2.5 upper=0 effort=500 velocity=0.2
- joint forearm_rotation: limit lower=-0.90 upper=1.3963 effort=50 velocity=8.3776 -> lower=-0.90 upper=1.3963 effort=500 velocity=1.2
- joint shoulder_rotation: limit lower=-3.14 upper=3.14 effort=1.8 velocity=8.3776 -> lower=-3.14 upper=3.14 effort=20 velocity=8.3776
- joint wrist_rotation: limit lower=-3.14 upper=3.14 effort=1.8 velocity=8.3776 -> lower=-3.14 upper=3.14 effort=18 velocity=8.3776

Commit message: Added velocity controller

File: Simulation/src/manipulator/urdf/manipulator.urdf (robot description, URDF)
Before this commit: robot manipulator, 8 links, 7 joints
Joints:
- joint shoulder_rotation: limit lower=-3.14 upper=3.14 effort=20 velocity=8.3776 -> lower=-3.14 upper=3.14 effort=50 velocity=8.3776
