Commit message: Simulation: add new controllers

File: Simulation/src/manipulator/urdf/manipulator_velocity.urdf (robot description, URDF)
Before this commit: robot manipulator, 8 links, 7 joints
Joints:
- joint arm_rotation: limit lower=-2.5 upper=0 effort=500 velocity=0.2 -> lower=-2.5 upper=0 effort=1000 velocity=0.2
- joint forearm_rotation: limit lower=-0.90 upper=1.3963 effort=500 velocity=1.2 -> lower=-0.90 upper=1.3963 effort=1000 velocity=1.2
- joint shoulder_rotation: limit lower=-3.14 upper=3.14 effort=50 velocity=8.3776 -> lower=-3.14 upper=3.14 effort=10 velocity=8.3776
- joint wrist_rotation: limit lower=-3.14 upper=3.14 effort=18 velocity=8.3776 -> lower=-3.14 upper=3.14 effort=36 velocity=8.3776
