Commit message: Simulation: experiments

File: Simulation/src/manipulator/urdf/manipulator_effort.urdf (robot description, URDF)
Before this commit: robot manipulator, 8 links, 7 joints
Joints:
- joint forearm_rotation: axis 0 0 -1 -> 0 0 1

Commit message: Add trajectory planning

File: Simulation/src/manipulator/urdf/manipulator_effort.urdf (robot description, URDF)
Before this commit: robot manipulator, 8 links, 7 joints
Joints:
- joint forearm_rotation: limit lower=-0.90 upper=1.3963 effort=1000 velocity=1.2 -> lower=-0.90 upper=1.3963 effort=2000 velocity=1.2
- joint gripper_rotation: limit lower=-3.14 upper=3.14 effort=10.8 velocity=5.236 -> lower=-3.14 upper=3.14 effort=21.6 velocity=5.236
- joint shoulder_rotation: limit lower=-3.14 upper=3.14 effort=10 velocity=8.3776 -> lower=-3.14 upper=3.14 effort=50 velocity=8.3776
- joint wrist_pitch: limit lower=0 upper=3.14 effort=10.8 velocity=5.236 -> lower=0 upper=3.14 effort=21.6 velocity=5.236
- joint wrist_rotation: limit lower=-3.14 upper=3.14 effort=36 velocity=8.3776 -> lower=-3.14 upper=3.14 effort=54 velocity=8.3776

File: Simulation/src/manipulator/urdf/manipulator_velocity.urdf (robot description, URDF)
Before this commit: robot manipulator, 8 links, 7 joints
Joints:
- joint forearm_rotation: limit lower=-0.90 upper=1.3963 effort=1000 velocity=1.2 -> lower=-0.90 upper=1.3963 effort=2000 velocity=1.2
- joint gripper_rotation: limit lower=-3.14 upper=3.14 effort=10.8 velocity=5.236 -> lower=-3.14 upper=3.14 effort=21.6 velocity=5.236
- joint shoulder_rotation: limit lower=-3.14 upper=3.14 effort=10 velocity=8.3776 -> lower=-3.14 upper=3.14 effort=50 velocity=8.3776
- joint wrist_pitch: limit lower=0 upper=3.14 effort=10.8 velocity=5.236 -> lower=0 upper=3.14 effort=21.6 velocity=5.236
- joint wrist_rotation: limit lower=-3.14 upper=3.14 effort=36 velocity=8.3776 -> lower=-3.14 upper=3.14 effort=54 velocity=8.3776

Commit message: Simulation: prepared simulation for tests

File: Simulation/src/manipulator/urdf/manipulator_effort.urdf (robot description, URDF)
Before this commit: robot manipulator, 8 links, 7 joints
Joints:
- joint arm_rotation: limit lower=-2.5 upper=0 effort=1000 velocity=0.2 -> lower=-2.5 upper=0 effort=1000 velocity=1.2; origin xyz=0 0.6 0 rpy=0 0 -1.3089 -> xyz=0 0.6 0 rpy=0 0 -1.2

File: Simulation/src/manipulator/urdf/manipulator_velocity.urdf (robot description, URDF)
Before this commit: robot manipulator, 8 links, 7 joints
Joints:
- joint arm_rotation: origin xyz=0 0.6 0 rpy=0 0 -1.3089 -> xyz=0 0.6 0 rpy=0 0 -1.2

Commit message: Finished writing line, circle, square tests

File: Simulation/src/manipulator/urdf/manipulator_effort.urdf (robot description, URDF)
Before this commit: robot manipulator, 8 links, 7 joints
Joints:
- joint arm_rotation: limit lower=-2.5 upper=0 effort=1000 velocity=1.2 -> lower=-2.5 upper=0 effort=2000 velocity=1.2
- joint shoulder_rotation: limit lower=-3.14 upper=3.14 effort=50 velocity=8.3776 -> lower=-3.14 upper=3.14 effort=50 velocity=2.3776
- joint wrist_rotation: limit lower=-3.14 upper=3.14 effort=54 velocity=8.3776 -> lower=-3.14 upper=3.14 effort=54 velocity=2.3776
